File: adapter/passive-3/passive3-rpi-hub75-adapter.kicad_pcb (KiCad board)
At the start: 2 copper layers, 80 x 23 mm, 6 parts, among them P1 CONN_02X20, P2 CONN_01X01, P3 CONN_01X01

Commit message: o update text.
Other:
- board text added: "github.com/hzeller/rpi-rgb-led-matrix"
- board text removed: "github.com/hzeller/rpi-rgb-led-matrix (v2)"
